Commit message: cpp init planning_scene checking if state is_valid and if ikfound

File: install/four_drone_demo/share/four_drone_demo/config/isaac_twin.ros2_control.xacro (robot description, xacro)
@@ -10,4 +10,5 @@
             <joint name="spherical_1_x">
                 <command_interface name="position"/>
+                <command_interface name="velocity"/>
                 <state_interface name="position">
                   <param name="initial_value">${initial_positions['spherical_1_x']}</param>
@@ -17,4 +18,5 @@
             <joint name="spherical_1_y">
                 <command_interface name="position"/>
+                <command_interface name="velocity"/>
                 <state_interface name="position">
                   <param name="initial_value">${initial_positions['spherical_1_y']}</param>
@@ -24,4 +26,5 @@
             <joint name="spherical_1_z">
                 <command_interface name="position"/>
+                <command_interface name="velocity"/>
                 <state_interface name="position">
                   <param name="initial_value">${initial_positions['spherical_1_z']}</param>
@@ -31,4 +34,5 @@
             <joint name="prismatic_joint_1">
                 <command_interface name="position"/>
+                <command_interface name="velocity"/>
                 <state_interface name="position">
                   <param name="initial_value">${initial_positions['prismatic_joint_1']}</param>
@@ -38,4 +42,5 @@
             <joint name="spherical_2_x">
                 <command_interface name="position"/>
+                <command_interface name="velocity"/>
                 <state_interface name="position">
                   <param name="initial_value">${initial_positions['spherical_2_x']}</param>
@@ -45,4 +50,5 @@
             <joint name="spherical_2_y">
                 <command_interface name="position"/>
+                <command_interface name="velocity"/>
                 <state_interface name="position">
                   <param name="initial_value">${initial_positions['spherical_2_y']}</param>
@@ -52,4 +58,5 @@
             <joint name="spherical_2_z">
                 <command_interface name="position"/>
+                <command_interface name="velocity"/>
                 <state_interface name="position">
                   <param name="initial_value">${initial_positions['spherical_2_z']}</param>
@@ -59,4 +66,5 @@
             <joint name="prismatic_joint_2">
                 <command_interface name="position"/>
+                <command_interface name="velocity"/>
                 <state_interface name="position">
                   <param name="initial_value">${initial_positions['prismatic_joint_2']}</param>
@@ -66,4 +74,5 @@
             <joint name="spherical_3_x">
                 <command_interface name="position"/>
+                <command_interface name="velocity"/>
                 <state_interface name="position">
                   <param name="initial_value">${initial_positions['spherical_3_x']}</param>
@@ -73,4 +82,5 @@
             <joint name="spherical_3_y">
                 <command_interface name="position"/>
+                <command_interface name="velocity"/>
                 <state_interface name="position">
                   <param name="initial_value">${initial_positions['spherical_3_y']}</param>
@@ -80,4 +90,5 @@
             <joint name="spherical_3_z">
                 <command_interface name="position"/>
+                <command_interface name="velocity"/>
                 <state_interface name="position">
                   <param name="initial_value">${initial_positions['spherical_3_z']}</param>
@@ -87,4 +98,5 @@
             <joint name="prismatic_joint_3">
                 <command_interface name="position"/>
+                <command_interface name="velocity"/>
                 <state_interface name="position">
                   <param name="initial_value">${initial_positions['prismatic_joint_3']}</param>
@@ -94,4 +106,5 @@
             <joint name="spherical_4_x">
                 <command_interface name="position"/>
+                <command_interface name="velocity"/>
                 <state_interface name="position">
                   <param name="initial_value">${initial_positions['spherical_4_x']}</param>
@@ -101,4 +114,5 @@
             <joint name="spherical_4_y">
                 <command_interface name="position"/>
+                <command_interface name="velocity"/>
                 <state_interface name="position">
                   <param name="initial_value">${initial_positions['spherical_4_y']}</param>
@@ -108,4 +122,5 @@
             <joint name="spherical_4_z">
                 <command_interface name="position"/>
+                <command_interface name="velocity"/>
                 <state_interface name="position">
                   <param name="initial_value">${initial_positions['spherical_4_z']}</param>
@@ -115,4 +130,5 @@
             <joint name="prismatic_joint_4">
                 <command_interface name="position"/>
+                <command_interface name="velocity"/>
                 <state_interface name="position">
                   <param name="initial_value">${initial_positions['prismatic_joint_4']}</param>

File: install/isaac_sim_demo/share/isaac_sim_demo/urdf/4_drones.urdf (robot description, URDF)
Before this commit: robot isaac_twin, 17 links, 16 joints
Links:
- link Drone1: geometry collision box size=0.25 0.25 0.25; visual box size=0.25 0.25 0.25
- link Drone2: geometry collision box size=0.25 0.25 0.25; visual box size=0.25 0.25 0.25
- link Drone3: geometry collision box size=0.25 0.25 0.25; visual box size=0.25 0.25 0.25
- link Drone4: geometry collision box size=0.25 0.25 0.25; visual box size=0.25 0.25 0.25
- link base_link: geometry visual box size=0.01 0.01 0
- link spherical_1_x: geometry visual box size=0.01 0.01 0
- link spherical_1_y: geometry visual box size=0.01 0.01 0
- link spherical_1_z: geometry visual box size=0.01 0.01 0
- link spherical_2_x: geometry visual box size=0.01 0.01 0
- link spherical_2_y: geometry visual box size=0.01 0.01 0
- link spherical_2_z: geometry visual box size=0.01 0.01 0
- link spherical_3_x: geometry visual box size=0.01 0.01 0
- link spherical_3_y: geometry visual box size=0.01 0.01 0
- link spherical_3_z: geometry visual box size=0.01 0.01 0
- link spherical_4_x: geometry visual box size=0.01 0.01 0
- link spherical_4_y: geometry visual box size=0.01 0.01 0
- link spherical_4_z: geometry visual box size=0.01 0.01 0
Joints:
- joint prismatic_joint_1: limit lower=0 upper=3 effort=10 velocity=1.0 -> lower=0 upper=4 effort=10 velocity=1.0; origin xyz=0 0 0 rpy=0 0 0 -> xyz=0 0 0.05 rpy=0 0 0
- joint prismatic_joint_2: limit lower=0 upper=3 effort=10 velocity=1.0 -> lower=0 upper=4 effort=10 velocity=1.0
- joint prismatic_joint_3: limit lower=0 upper=3 effort=10 velocity=1.0 -> lower=0 upper=4 effort=10 velocity=1.0
- joint prismatic_joint_4: limit lower=0 upper=3 effort=10 velocity=1.0 -> lower=0 upper=4 effort=10 velocity=1.0
- joint spherical_1_x: limit lower=-1.57 upper=1.57 effort=10 velocity=1.0 -> (none); type revolute -> continuous
- joint spherical_1_y: limit lower=-1.57 upper=1.57 effort=10 velocity=1.0 -> (none); origin xyz=0 0 0 rpy=0 0 0 -> xyz=0 0 0 rpy=0 0 1.570; type revolute -> continuous
- joint spherical_2_x: limit lower=-1.57 upper=1.57 effort=10 velocity=1.0 -> (none); type revolute -> continuous
- joint spherical_2_y: limit lower=-1.57 upper=1.57 effort=10 velocity=1.0 -> (none); type revolute -> continuous
- joint spherical_3_x: limit lower=-1.57 upper=1.57 effort=10 velocity=1.0 -> (none); type revolute -> continuous
- joint spherical_3_y: limit lower=-1.57 upper=1.57 effort=10 velocity=1.0 -> (none); type revolute -> continuous
- joint spherical_4_x: limit lower=-1.57 upper=1.57 effort=10 velocity=1.0 -> (none); type revolute -> continuous
- joint spherical_4_y: limit lower=-1.57 upper=1.57 effort=10 velocity=1.0 -> (none); type revolute -> continuous

File: install/isaac_sim_demo/share/isaac_sim_demo/urdf/4_drones.xacro (robot description, xacro)
@@ -19,9 +19,9 @@
     <parent link="spherical_1_z"/>
     <child link="Drone1"/>
-    <origin xyz="0 0 0" rpy="0 0 0"/>
+    <origin xyz="0 0 0.0" rpy="0 0 0"/>
     <axis xyz="0 0 1"/>
     <limit lower="0" upper="3" effort="10" velocity="1.0"/>
   </joint>
-  <xacro:temp_link name="Drone1" origin_xyz="0 0 0" origin_rpy="0 0 0" size="0.1 0.1 0.1" mass="0.1" />
+  <xacro:temp_link name="Drone1" origin_xyz="0 0 0" origin_rpy="0 0 0" size="0.3 0.3 0.1" mass="0.1" />
   <xacro:spherical_joint prefix="spherical_2" parent="Drone1" />
   <joint name="prismatic_joint_2" type="prismatic">
@@ -32,5 +32,5 @@
     <limit lower="0" upper="3" effort="10" velocity="1.0"/>
   </joint>
-  <xacro:temp_link name="Drone2" origin_xyz="0 0 0" origin_rpy="0 0 0" size="0.1 0.1 0.1" mass="0.1" />
+  <xacro:temp_link name="Drone2" origin_xyz="0 0 0" origin_rpy="0 0 0" size="0.3 0.3 0.1" mass="0.1" />
   <xacro:spherical_joint prefix="spherical_3" parent="Drone2" />
   <joint name="prismatic_joint_3" type="prismatic">
@@ -41,5 +41,5 @@
     <limit lower="0" upper="3" effort="10" velocity="1.0"/>
   </joint>
-  <xacro:temp_link name="Drone3" origin_xyz="0 0 0" origin_rpy="0 0 0" size="0.1 0.1 0.1" mass="0.1" />
+  <xacro:temp_link name="Drone3" origin_xyz="0 0 0" origin_rpy="0 0 0" size="0.3 0.3 0.1" mass="0.1" />
   <xacro:spherical_joint prefix="spherical_4" parent="Drone3" />
   <joint name="prismatic_joint_4" type="prismatic">

File: install/isaac_sim_demo/share/isaac_sim_demo/urdf/chain.xacro (robot description, xacro)
@@ -3,11 +3,11 @@
   <!-- Define parameters -->
   <xacro:property name="cylinder_radius" value="0.01"/>
-  <xacro:property name="cylinder_length" value="0.05"/>
+  <xacro:property name="cylinder_length" value="0.1"/>
   <xacro:property name="num_links" value="20"/>
   <!-- Macro for Chain Links -->
-  <xacro:macro name="chain" params="parent_link child_link">
+  <xacro:macro name="chain" params="parent_link child_link prefix">
     <!-- Define the chain starting from the parent link -->
     <xacro:macro name="chain_link" params="index parent_link remaining_links">
-      <link name="link_${index}">
+      <link name="${prefix}_link_${index}">
         <visual>
           <origin xyz="0 0 0" rpy="0 0 0"/>
@@ -19,8 +19,14 @@
           </material>
         </visual>
+      <collision>
+        <origin xyz="0 0 0" rpy="0 0 0" />
+        <geometry>
+           <cylinder radius="${cylinder_radius}" length="${cylinder_length}"/>
+        </geometry>
+      </collision>
       </link>
-      <joint name="joint_${index}" type="continuous">
+      <joint name="${prefix}_joint_${index}" type="continuous">
         <parent link="${parent_link}"/>
-        <child link="link_${index}"/>
+        <child link="${prefix}_link_${index}"/>
         <origin xyz="0 0 ${cylinder_length / 2}" rpy="0 0 0"/>
         <axis xyz="0 0 1"/>
@@ -28,5 +34,5 @@
       <!-- Recursively create the next link if there are remaining links -->
       <xacro:if value="${remaining_links > 0}">
-        <xacro:chain_link index="${index + 1}" parent_link="link_${index}" remaining_links="${remaining_links - 1}"/>
+        <xacro:chain_link index="${index + 1}" parent_link="${prefix}_link_${index}" remaining_links="${remaining_links - 1}"/>
       </xacro:if>
     </xacro:macro>
@@ -34,6 +40,6 @@
     <xacro:chain_link index="1" parent_link="${parent_link}" remaining_links="${num_links - 2}"/>
     <!-- Define the final joint to the child link -->
-    <joint name="joint_${num_links}" type="continuous">
-      <parent link="link_${num_links - 1}"/>
+    <joint name="${prefix}_joint_${num_links}" type="continuous">
+      <parent link="${prefix}_link_${num_links - 1}"/>
       <child link="${child_link}"/>
       <origin xyz="0 0 ${cylinder_length / 2}" rpy="0 0 0"/>

File: install/isaac_sim_demo/share/isaac_sim_demo/urdf/two_drones.urdf (robot description, URDF)
Before this commit: robot isaac_twin, 9 links, 8 joints
Links:
- removed link spherical_1_x
- removed link spherical_1_y
- removed link spherical_1_z
- removed link spherical_2_x
- removed link spherical_2_y
- removed link spherical_2_z
Joints:
- removed joint prismatic_joint_1
- removed joint prismatic_joint_2
- removed joint spherical_1_x
- removed joint spherical_1_y
- removed joint spherical_1_z
- removed joint spherical_2_x
- removed joint spherical_2_y
- removed joint spherical_2_z
- added joint floating_1: type floating, parent base_link, child Drone1, origin xyz=0 0 0.0 rpy=0 0 0, axis 1 0 0
- added joint floating_2: type floating, parent Drone1, child Drone2, origin xyz=0 0 0.0 rpy=0 0 0, axis 1 0 0

File: install/test_moveit_config/share/test_moveit_config/config/isaac_twin.ros2_control.xacro (robot description, xacro)
@@ -10,4 +10,5 @@
             <joint name="spherical_1_x">
                 <command_interface name="position"/>
+                <command_interface name="velocity"/>
                 <state_interface name="position">
                   <param name="initial_value">${initial_positions['spherical_1_x']}</param>
@@ -17,4 +18,5 @@
             <joint name="spherical_1_y">
                 <command_interface name="position"/>
+                <command_interface name="velocity"/>
                 <state_interface name="position">
                   <param name="initial_value">${initial_positions['spherical_1_y']}</param>
@@ -24,4 +26,5 @@
             <joint name="spherical_1_z">
                 <command_interface name="position"/>
+                <command_interface name="velocity"/>
                 <state_interface name="position">
                   <param name="initial_value">${initial_positions['spherical_1_z']}</param>
@@ -29,13 +32,7 @@
                 <state_interface name="velocity"/>
             </joint>
-            <joint name="prismatic_joint_1">
-                <command_interface name="position"/>
-                <state_interface name="position">
-                  <param name="initial_value">${initial_positions['prismatic_joint_1']}</param>
-                </state_interface>
-                <state_interface name="velocity"/>
-            </joint>
             <joint name="spherical_2_x">
                 <command_interface name="position"/>
+                <command_interface name="velocity"/>
                 <state_interface name="position">
                   <param name="initial_value">${initial_positions['spherical_2_x']}</param>
@@ -45,4 +42,5 @@
             <joint name="spherical_2_y">
                 <command_interface name="position"/>
+                <command_interface name="velocity"/>
                 <state_interface name="position">
                   <param name="initial_value">${initial_positions['spherical_2_y']}</param>
@@ -52,4 +50,5 @@
             <joint name="spherical_2_z">
                 <command_interface name="position"/>
+                <command_interface name="velocity"/>
                 <state_interface name="position">
                   <param name="initial_value">${initial_positions['spherical_2_z']}</param>
@@ -57,8 +56,49 @@
                 <state_interface name="velocity"/>
             </joint>
-            <joint name="prismatic_joint_2">
+            <joint name="spherical_3_x">
                 <command_interface name="position"/>
+                <command_interface name="velocity"/>
                 <state_interface name="position">
-                  <param name="initial_value">${initial_positions['prismatic_joint_2']}</param>
+                  <param name="initial_value">${initial_positions['spherical_3_x']}</param>
+                </state_interface>
+                <state_interface name="velocity"/>
+            </joint>
+            <joint name="spherical_3_y">
+                <command_interface name="position"/>
+                <command_interface name="velocity"/>
+                <state_interface name="position">
+                  <param name="initial_value">${initial_positions['spherical_3_y']}</param>
+                </state_interface>
+                <state_interface name="velocity"/>
+            </joint>
+            <joint name="spherical_3_z">
+                <command_interface name="position"/>
+                <command_interface name="velocity"/>
+                <state_interface name="position">
+                  <param name="initial_value">${initial_positions['spherical_3_z']}</param>
+                </state_interface>
+                <state_interface name="velocity"/>
+            </joint>
+            <joint name="spherical_4_x">
+                <command_interface name="position"/>
+                <command_interface name="velocity"/>
+                <state_interface name="position">
+                  <param name="initial_value">${initial_positions['spherical_4_x']}</param>
+                </state_interface>
+                <state_interface name="velocity"/>
+            </joint>
+            <joint name="spherical_4_y">
+                <command_interface name="position"/>
+                <command_interface name="velocity"/>
+                <state_interface name="position">
+                  <param name="initial_value">${initial_positions['spherical_4_y']}</param>
+                </state_interface>
+                <state_interface name="velocity"/>
+            </joint>
+            <joint name="spherical_4_z">
+                <command_interface name="position"/>
+                <command_interface name="velocity"/>
+                <state_interface name="position">
+                  <param name="initial_value">${initial_positions['spherical_4_z']}</param>
                 </state_interface>
                 <state_interface name="velocity"/>

File: install/test_moveit_config/share/test_moveit_config/config/isaac_twin.urdf.xacro (robot description, xacro)
@@ -3,5 +3,5 @@
     <xacro:arg name="initial_positions_file" default="initial_positions.yaml" />
     <!-- Import isaac_twin urdf file -->
-    <xacro:include filename="$(find isaac_sim_demo)/urdf/two_drones.urdf" />
+    <xacro:include filename="$(find isaac_sim_demo)/urdf/chain_twin.urdf" />
     <!-- Import control_xacro -->
     <xacro:include filename="isaac_twin.ros2_control.xacro" />
