Commit message: bullet line of sight

File: src/isaac_sim_demo/urdf/4_drones_copy_2.urdf (robot description, URDF)
Before this commit: robot isaac_twin, 13 links, 12 joints
Links:
- added link spherical_1_z, mass 0.1; visual box size=0.01 0.01 0
- added link spherical_2_z, mass 0.1; visual box size=0.01 0.01 0
- added link spherical_3_z, mass 0.1; visual box size=0.01 0.01 0
- added link spherical_4_z, mass 0.1; visual box size=0.01 0.01 0
Joints:
- added joint prismatic_joint_1: type prismatic, parent spherical_1_z, child Drone1, origin xyz=0 0 0.05 rpy=0 0 0, axis 0 0 1, limit lower=0 upper=4 effort=10 velocity=1.0
- added joint prismatic_joint_2: type prismatic, parent spherical_2_z, child Drone2, origin xyz=0 0 0 rpy=0 0 0, axis 0 0 1, limit lower=0 upper=4 effort=10 velocity=1.0
- added joint prismatic_joint_3: type prismatic, parent spherical_3_z, child Drone3, origin xyz=0 0 0 rpy=0 0 0, axis 0 0 1, limit lower=0 upper=4 effort=10 velocity=1.0
- added joint prismatic_joint_4: type prismatic, parent spherical_4_z, child Drone4, origin xyz=0 0 0 rpy=0 0 0, axis 0 0 1, limit lower=0 upper=4 effort=10 velocity=1.0
- joint spherical_1_x: limit lower=0 upper=4 effort=10 velocity=1.0 -> (none); type prismatic -> continuous
- joint spherical_1_y: limit lower=0 upper=4 effort=10 velocity=1.0 -> (none); type prismatic -> continuous
- joint spherical_1_z: child Drone1 -> spherical_1_z; limit lower=0 upper=4 effort=10 velocity=1.0 -> (none); origin xyz=0 0 0 rpy=0 0 -1.5354 -> xyz=0 0 0 rpy=0 0 0; type prismatic -> continuous
- joint spherical_2_x: limit lower=0 upper=4 effort=10 velocity=1.0 -> (none); type prismatic -> continuous
- joint spherical_2_y: limit lower=0 upper=4 effort=10 velocity=1.0 -> (none); type prismatic -> continuous
- joint spherical_2_z: child Drone2 -> spherical_2_z; limit lower=0 upper=4 effort=10 velocity=1.0 -> (none); type prismatic -> continuous
- joint spherical_3_x: limit lower=0 upper=4 effort=10 velocity=1.0 -> (none); type prismatic -> continuous
- joint spherical_3_y: limit lower=0 upper=4 effort=10 velocity=1.0 -> (none); type prismatic -> continuous
- joint spherical_3_z: child Drone3 -> spherical_3_z; limit lower=0 upper=4 effort=10 velocity=1.0 -> (none); type prismatic -> continuous
- joint spherical_4_x: limit lower=0 upper=4 effort=10 velocity=1.0 -> (none); type prismatic -> continuous
- joint spherical_4_y: limit lower=0 upper=4 effort=10 velocity=1.0 -> (none); type prismatic -> continuous
- joint spherical_4_z: child Drone4 -> spherical_4_z; limit lower=0 upper=4 effort=10 velocity=1.0 -> (none); type prismatic -> continuous
