Commit message: v1.0

File: src/isaac_sim_demo/urdf/4_drones.urdf (robot description, URDF)
Before this commit: robot isaac_twin, 13 links, 12 joints
Joints:
- joint spherical_1_x: limit lower=0 upper=4 effort=10 velocity=1.0 -> lower=-4 upper=4 effort=10 velocity=1.0
- joint spherical_1_y: limit lower=0 upper=4 effort=10 velocity=1.0 -> lower=-4 upper=4 effort=10 velocity=1.0
- joint spherical_1_z: limit lower=0 upper=4 effort=10 velocity=1.0 -> lower=-4 upper=4 effort=10 velocity=1.0
- joint spherical_2_x: limit lower=0 upper=4 effort=10 velocity=1.0 -> lower=-4 upper=4 effort=10 velocity=1.0
- joint spherical_2_y: limit lower=0 upper=4 effort=10 velocity=1.0 -> lower=-4 upper=4 effort=10 velocity=1.0
- joint spherical_2_z: limit lower=0 upper=4 effort=10 velocity=1.0 -> lower=-4 upper=4 effort=10 velocity=1.0
- joint spherical_3_x: limit lower=0 upper=4 effort=10 velocity=1.0 -> lower=-4 upper=4 effort=10 velocity=1.0
- joint spherical_3_y: limit lower=0 upper=4 effort=10 velocity=1.0 -> lower=-4 upper=4 effort=10 velocity=1.0
- joint spherical_3_z: limit lower=0 upper=4 effort=10 velocity=1.0 -> lower=-4 upper=4 effort=10 velocity=1.0
- joint spherical_4_x: limit lower=0 upper=4 effort=10 velocity=1.0 -> lower=-4 upper=4 effort=10 velocity=1.0
- joint spherical_4_y: limit lower=0 upper=4 effort=10 velocity=1.0 -> lower=-4 upper=4 effort=10 velocity=1.0
- joint spherical_4_z: limit lower=0 upper=4 effort=10 velocity=1.0 -> lower=-4 upper=4 effort=10 velocity=1.0

Commit message: Update 4_drones.urdf

File: src/isaac_sim_demo/urdf/4_drones.urdf (robot description, URDF)
Before this commit: robot isaac_twin, 13 links, 12 joints
Links:
- link Drone1: geometry collision box size=0.6 0.6 0.2; visual box size=0.6 0.6 0.2
- link Drone2: geometry collision box size=0.6 0.6 0.2; visual box size=0.6 0.6 0.2
- link Drone3: geometry collision box size=0.6 0.6 0.2; visual box size=0.6 0.6 0.2
- link Drone4: geometry collision box size=0.6 0.6 0.2; visual box size=0.6 0.6 0.2

Commit message: Update 4_drones.urdf

File: src/isaac_sim_demo/urdf/4_drones.urdf (robot description, URDF)
Before this commit: robot isaac_twin, 13 links, 12 joints
Links:
- link Drone1: geometry collision box size=0.65 0.65 0.25; visual box size=0.65 0.65 0.25
- link Drone2: geometry collision box size=0.65 0.65 0.25; visual box size=0.65 0.65 0.25
- link Drone3: geometry collision box size=0.65 0.65 0.25; visual box size=0.6 0.6 0.25
- link Drone4: geometry collision box size=0.65 0.65 0.25; visual box size=0.65 0.65 0.25
