Commit message: v1.0

File: install/isaac_sim_demo/share/isaac_sim_demo/urdf/4_drones.urdf (robot description, URDF)
Before this commit: robot isaac_twin, 17 links, 16 joints
Links:
- removed link spherical_1_z
- removed link spherical_2_z
- removed link spherical_3_z
- removed link spherical_4_z
- link Drone1: geometry collision box size=0.3 0.3 0.3; visual box size=0.3 0.3 0.3
- link Drone2: geometry collision box size=0.3 0.3 0.3; visual box size=0.3 0.3 0.3
- link Drone3: geometry collision box size=0.3 0.3 0.3; visual box size=0.3 0.3 0.3
- link Drone4: geometry collision box size=0.3 0.3 0.3; visual box size=0.3 0.3 0.3
Joints:
- removed joint prismatic_joint_1
- removed joint prismatic_joint_2
- removed joint prismatic_joint_3
- removed joint prismatic_joint_4
- joint spherical_1_x: limit (none) -> lower=-4 upper=4 effort=10 velocity=1.0; type continuous -> prismatic
- joint spherical_1_y: limit (none) -> lower=-4 upper=4 effort=10 velocity=1.0; origin xyz=0 0 0 rpy=0 0 1.570 -> xyz=0 0 0 rpy=0 0 0; type continuous -> prismatic
- joint spherical_1_z: child spherical_1_z -> Drone1; limit (none) -> lower=-4 upper=4 effort=10 velocity=1.0; origin xyz=0 0 0 rpy=0 0 0 -> xyz=0 0 0 rpy=0 0 -1.5354; type continuous -> prismatic
- joint spherical_2_x: limit (none) -> lower=-4 upper=4 effort=10 velocity=1.0; type continuous -> prismatic
- joint spherical_2_y: limit (none) -> lower=-4 upper=4 effort=10 velocity=1.0; type continuous -> prismatic
- joint spherical_2_z: child spherical_2_z -> Drone2; limit (none) -> lower=-4 upper=4 effort=10 velocity=1.0; type continuous -> prismatic
- joint spherical_3_x: limit (none) -> lower=-4 upper=4 effort=10 velocity=1.0; type continuous -> prismatic
- joint spherical_3_y: limit (none) -> lower=-4 upper=4 effort=10 velocity=1.0; type continuous -> prismatic
- joint spherical_3_z: child spherical_3_z -> Drone3; limit (none) -> lower=-4 upper=4 effort=10 velocity=1.0; type continuous -> prismatic
- joint spherical_4_x: limit (none) -> lower=-4 upper=4 effort=10 velocity=1.0; type continuous -> prismatic
- joint spherical_4_y: limit (none) -> lower=-4 upper=4 effort=10 velocity=1.0; type continuous -> prismatic
- joint spherical_4_z: child spherical_4_z -> Drone4; limit (none) -> lower=-4 upper=4 effort=10 velocity=1.0; type continuous -> prismatic
