Commit message: final

File: install/isaac_sim_demo/share/isaac_sim_demo/urdf/4_drones copy.urdf (robot description, URDF)
Before this commit: robot isaac_twin, 17 links, 16 joints
Links:
- removed link spherical_1_z
- removed link spherical_2_z
- removed link spherical_3_z
- removed link spherical_4_z
- link Drone1: geometry collision box size=0.65 0.65 0.25; visual box size=0.65 0.65 0.25
- link Drone2: geometry collision box size=0.65 0.65 0.25; visual box size=0.65 0.65 0.25
- link Drone3: geometry collision box size=0.65 0.65 0.25; visual box size=0.65 0.65 0.25
- link Drone4: geometry collision box size=0.65 0.65 0.25; visual box size=0.65 0.65 0.25
- link base_link: geometry visual box size=0.01 0.01 0
- link spherical_1_x: geometry visual box size=0.01 0.01 0
- link spherical_1_y: geometry visual box size=0.01 0.01 0
- link spherical_2_x: geometry visual box size=0.01 0.01 0
- link spherical_2_y: geometry visual box size=0.01 0.01 0
- link spherical_3_x: geometry visual box size=0.01 0.01 0
- link spherical_3_y: geometry visual box size=0.01 0.01 0
- link spherical_4_x: geometry visual box size=0.01 0.01 0
- link spherical_4_y: geometry visual box size=0.01 0.01 0
Joints:
- removed joint prismatic_joint_1
- removed joint prismatic_joint_2
- removed joint prismatic_joint_3
- removed joint prismatic_joint_4
- joint spherical_1_x: limit lower=-1.57 upper=1.57 effort=10 velocity=1.0 -> lower=-4 upper=4 effort=10 velocity=1.0; type revolute -> prismatic
- joint spherical_1_y: limit lower=-1.57 upper=1.57 effort=10 velocity=1.0 -> lower=-4 upper=4 effort=10 velocity=1.0; type revolute -> prismatic
- joint spherical_1_z: child spherical_1_z -> Drone1; limit (none) -> lower=-4 upper=4 effort=10 velocity=1.0; origin xyz=0 0 0 rpy=0 0 0 -> xyz=0 0 0 rpy=0 0 -1.5354; type continuous -> prismatic
- joint spherical_2_x: limit lower=-1.57 upper=1.57 effort=10 velocity=1.0 -> lower=-4 upper=4 effort=10 velocity=1.0; type revolute -> prismatic
- joint spherical_2_y: limit lower=-1.57 upper=1.57 effort=10 velocity=1.0 -> lower=-4 upper=4 effort=10 velocity=1.0; type revolute -> prismatic
- joint spherical_2_z: child spherical_2_z -> Drone2; limit (none) -> lower=-4 upper=4 effort=10 velocity=1.0; type continuous -> prismatic
- joint spherical_3_x: limit lower=-1.57 upper=1.57 effort=10 velocity=1.0 -> lower=-4 upper=4 effort=10 velocity=1.0; type revolute -> prismatic
- joint spherical_3_y: limit lower=-1.57 upper=1.57 effort=10 velocity=1.0 -> lower=-4 upper=4 effort=10 velocity=1.0; type revolute -> prismatic
- joint spherical_3_z: child spherical_3_z -> Drone3; limit (none) -> lower=-4 upper=4 effort=10 velocity=1.0; type continuous -> prismatic
- joint spherical_4_x: limit lower=-1.57 upper=1.57 effort=10 velocity=1.0 -> lower=-4 upper=4 effort=10 velocity=1.0; type revolute -> prismatic
- joint spherical_4_y: limit lower=-1.57 upper=1.57 effort=10 velocity=1.0 -> lower=-4 upper=4 effort=10 velocity=1.0; type revolute -> prismatic
- joint spherical_4_z: child spherical_4_z -> Drone4; limit (none) -> lower=-4 upper=4 effort=10 velocity=1.0; type continuous -> prismatic

File: install/isaac_sim_demo/share/isaac_sim_demo/urdf/4_drones.urdf (robot description, URDF)
Before this commit: robot isaac_twin, 13 links, 12 joints
Links:
- link Drone1: geometry collision box size=0.65 0.65 0.25; visual box size=0.65 0.65 0.25
- link Drone2: geometry collision box size=0.65 0.65 0.25; visual box size=0.65 0.65 0.25
- link Drone3: geometry collision box size=0.65 0.65 0.25; visual box size=0.65 0.65 0.25
- link Drone4: geometry collision box size=0.65 0.65 0.25; visual box size=0.65 0.65 0.25

File: install/isaac_sim_demo/share/isaac_sim_demo/urdf/4_drones_copy_2.urdf (robot description, URDF)
Before this commit: robot isaac_twin, 17 links, 16 joints
Links:
- removed link spherical_1_x
- removed link spherical_1_y
- removed link spherical_1_z
- removed link spherical_2_x
- removed link spherical_2_y
- removed link spherical_2_z
- removed link spherical_3_x
- removed link spherical_3_y
- removed link spherical_3_z
- removed link spherical_4_x
- removed link spherical_4_y
- removed link spherical_4_z
- added link prismatic_link_1_1, mass 0.1; visual box size=0.01 0.01 0
- added link prismatic_link_1_2, mass 0.1; visual box size=0.01 0.01 0
- added link prismatic_link_2_1, mass 0.1; visual box size=0.01 0.01 0
- added link prismatic_link_2_2, mass 0.1; visual box size=0.01 0.01 0
- added link prismatic_link_3_1, mass 0.1; visual box size=0.01 0.01 0
- added link prismatic_link_3_2, mass 0.1; visual box size=0.01 0.01 0
- added link prismatic_link_4_1, mass 0.1; visual box size=0.01 0.01 0
- added link prismatic_link_4_2, mass 0.1; visual box size=0.01 0.01 0
- link Drone1: geometry collision box size=0.65 0.65 0.25; visual box size=0.65 0.65 0.25
- link Drone2: geometry collision box size=0.65 0.65 0.25; visual box size=0.65 0.65 0.25
- link Drone3: geometry collision box size=0.65 0.65 0.25; visual box size=0.65 0.65 0.25
- link Drone4: geometry collision box size=0.65 0.65 0.25; visual box size=0.65 0.65 0.25
Joints:
- removed joint prismatic_joint_1
- removed joint prismatic_joint_2
- removed joint prismatic_joint_3
- removed joint prismatic_joint_4
- removed joint spherical_1_x
- removed joint spherical_1_y
- removed joint spherical_1_z
- removed joint spherical_2_x
- removed joint spherical_2_y
- removed joint spherical_2_z
- removed joint spherical_3_x
- removed joint spherical_3_y
- removed joint spherical_3_z
- removed joint spherical_4_x
- removed joint spherical_4_y
- removed joint spherical_4_z
- added joint prismatic_1_x: type prismatic, parent base_link, child prismatic_link_1_1, origin xyz=0 0 0.0 rpy=0 0 0, axis 1 0 0, limit lower=-4 upper=4 effort=10 velocity=1.0
- added joint prismatic_1_y: type prismatic, parent prismatic_link_1_1, child prismatic_link_1_2, origin xyz=0 0 0 rpy=0 0 0, axis 0 1 0, limit lower=-4 upper=4 effort=10 velocity=1.0
- added joint prismatic_1_z: type prismatic, parent prismatic_link_1_2, child Drone1, origin xyz=0 0 0 rpy=0 0 -1.5354, axis 0 0 1, limit lower=-4 upper=4 effort=10 velocity=1.0
- added joint prismatic_2_x: type prismatic, parent Drone1, child prismatic_link_2_1, origin xyz=0 0 0.0 rpy=0 0 0, axis 1 0 0, limit lower=-4 upper=4 effort=10 velocity=1.0
- added joint prismatic_2_y: type prismatic, parent prismatic_link_2_1, child prismatic_link_2_2, origin xyz=0 0 0 rpy=0 0 0, axis 0 1 0, limit lower=-4 upper=4 effort=10 velocity=1.0
- added joint prismatic_2_z: type prismatic, parent prismatic_link_2_2, child Drone2, origin xyz=0 0 0 rpy=0 0 0, axis 0 0 1, limit lower=-4 upper=4 effort=10 velocity=1.0
- added joint prismatic_3_x: type prismatic, parent Drone2, child prismatic_link_3_1, origin xyz=0 0 0.0 rpy=0 0 0, axis 1 0 0, limit lower=-4 upper=4 effort=10 velocity=1.0
- added joint prismatic_3_y: type prismatic, parent prismatic_link_3_1, child prismatic_link_3_2, origin xyz=0 0 0 rpy=0 0 0, axis 0 1 0, limit lower=-4 upper=4 effort=10 velocity=1.0
- added joint prismatic_3_z: type prismatic, parent prismatic_link_3_2, child Drone3, origin xyz=0 0 0 rpy=0 0 0, axis 0 0 1, limit lower=-4 upper=4 effort=10 velocity=1.0
- added joint prismatic_4_x: type prismatic, parent Drone3, child prismatic_link_4_1, origin xyz=0 0 0.0 rpy=0 0 0, axis 1 0 0, limit lower=-4 upper=4 effort=10 velocity=1.0
- added joint prismatic_4_y: type prismatic, parent prismatic_link_4_1, child prismatic_link_4_2, origin xyz=0 0 0 rpy=0 0 0, axis 0 1 0, limit lower=-4 upper=4 effort=10 velocity=1.0
- added joint prismatic_4_z: type prismatic, parent prismatic_link_4_2, child Drone4, origin xyz=0 0 0 rpy=0 0 0, axis 0 0 1, limit lower=-4 upper=4 effort=10 velocity=1.0
